File: variable_load.sch (KiCad schematic (older format))
At the start: 44 parts, among them Q1 NTD4858N, U1 LM324

Commit message: Revised
Parts:
- removed J?: Conn_01x03, symbol Conn_01x03
- removed JP? (x2): Jumper_NO_Small, symbol Jumper_NO_Small
- removed U?: LT1085-3.3, symbol LT1085-3.3
- added C23, C24: C, Capacitors_SMD:C_0805, symbol C
- added J2: Conn_01x04, Connectors_Molex:Molex_MiniFit-JR-5569-04A2_2x02x4.20mm_Angled, symbol Conn_01x04
- added J3: LEMO, variable_load:lemo_epb00250ntn, symbol LEMO
- added J6: GS3, Connectors:GS3, symbol GS3
- added R15, R16, R5, R6: R, Resistors_SMD:R_0805, symbol R
- added unit 3 of U2
- added unit 4 of U2
- added U3: TLV1117-33, TO_SOT_Packages_SMD:SOT-223-3_TabPin2, symbol TLV1117-33
- C1, C10, C11, C12, C13, C14, C15, C16, C17, C18, C19, C2, C20, C21, C22, C3, C4, C5, C6, C7, C8, C9: renamed from C?; footprint (none) -> Capacitors_SMD:C_0805
- J1, J4: renamed from J?; footprint (none) -> Pin_Headers:Pin_Header_Straight_1x02_Pitch2.54mm
- J5: renamed from J?; footprint (none) -> Connectors_Molex:Molex_MiniFit-JR-5569-04A2_2x02x4.20mm_Angled
- Q1: footprint TO_SOT_Packages_THT:TO-92_Molded_Narrow -> TO_SOT_Packages_SMD:TO-252-2
- R1, R13, R2, R3, R4, R7, R8: renamed from R?; footprint (none) -> Resistors_SMD:R_0805
- R10: renamed from R2; footprint (none) -> Resistors_SMD:R_0805
- R11: renamed from R3; footprint (none) -> Resistors_SMD:R_0805
- R12: renamed from R4; footprint (none) -> Resistors_SMD:R_0805
- R9: renamed from R1; footprint (none) -> Resistors_SMD:R_0805
- U2: renamed from U1; footprint (none) -> Housings_SOIC:SOIC-14_3.9x8.7mm_Pitch1.27mm
- gave numbers to parts that had none: 1
- renumbered R5 to R14
Connections:
- net labels added: 3V3LDO
- wire segments 103 -> 117
- no-connect marks 8 -> 7
Other:
- moved on the sheet: C10, C11, C12, C13, C15, C16, C17, C18, C19, C20, C22, C3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

Commit message: USB>I2C added
Parts:
- added C25, C26: C, Capacitors_SMD:C_0805, symbol C
- added J7: Conn_01x04, Connectors_Molex:Molex_MiniFit-JR-5569-04A2_2x02x4.20mm_Angled, symbol Conn_01x04
- added R17, R18, R19, R20: R, Resistors_SMD:R_0805, symbol R
- added U4: adafruit_ft232h, kk_adafruit:adafruit_ft232h_nohole, symbol adafruit_ft232h
- added U5: APD123, TO_SOT_Packages_SMD:SOT-23-5_HandSoldering, symbol APD123
Connections:
- net labels added: SCL, SDA, VREF
- wire segments 117 -> 149
- no-connect marks 7 -> 22
Other:
- moved on the sheet: U2C, U2D

Commit message: level shifter added
Parts:
- removed U5: APD123, TO_SOT_Packages_SMD:SOT-23-5_HandSoldering, symbol APD123
- added C27: C, Capacitors_SMD:C_0805, symbol C
- added J8: Conn_01x04, Connectors_Molex:Molex_MiniFit-JR-5569-04A2_2x02x4.20mm_Angled, symbol Conn_01x04
- added JP1, JP2: Jumper_NO_Small, Connectors:Banana_Jack_2Pin, symbol Jumper_NO_Small
- added R21, R22, R24, R25: R, Resistors_SMD:R_0805, symbol R
- added R23: 200k, Resistors_SMD:R_0805, symbol R
- added U5: PCA9306, Housings_SSOP:SSOP-8_2.95x2.8mm_Pitch0.65mm, symbol PCA9306
- added U6: APD123, TO_SOT_Packages_SMD:TSOT-23-5_HandSoldering, symbol APD123
- C25, C26: value C -> 1uF
Connections:
- net labels added: +Vcc, -Vcc, GNDREF, VCC_DAC, VCC_OPAMP, VREF1, V_DPU, Vcc
- wire segments 149 -> 173
- no-connect marks 22 -> 29
Other:
- moved on the sheet: C25, C26, R19, R20, U2C, U2D

Commit message: level shifter corrected footprint
Parts:
- JP1, JP2: footprint Connectors:Banana_Jack_2Pin -> Pin_Headers:Pin_Header_Angled_1x02_Pitch2.54mm
- U5: footprint Housings_SSOP:SSOP-8_2.95x2.8mm_Pitch0.65mm -> Housings_SSOP:VSSOP-8_2.3x2mm_Pitch0.5mm
Changed lines of the file:
@@
 F 0 "U5" H 8050 6150 50  0000 L CNN
 F 1 "PCA9306" H 8550 6150 50  0000 L CNN
-F 2 "Housings_SSOP:SSOP-8_2.95x2.8mm_Pitch0.65mm" H 7950 6050 50  0001 C CNN
+F 2 "Housings_SSOP:VSSOP-8_2.3x2mm_Pitch0.5mm" H 7950 6050 50  0001 C CNN
 F 3 "" H 8050 6150 50  0001 C CNN
 	1    8350 5700
@@
 F 0 "JP1" H 9900 5480 50  0000 C CNN
 F 1 "Jumper_NO_Small" H 9910 5340 50  0000 C CNN
-F 2 "Connectors:Banana_Jack_2Pin" H 9900 5400 50  0001 C CNN
+F 2 "Pin_Headers:Pin_Header_Angled_1x02_Pitch2.54mm" H 9900 5400 50  0001 C CNN
 F 3 "" H 9900 5400 50  0001 C CNN
 	1    9900 5400
@@
 F 0 "JP2" H 9900 5880 50  0000 C CNN
 F 1 "Jumper_NO_Small" H 9910 5740 50  0000 C CNN
-F 2 "Connectors:Banana_Jack_2Pin" H 9900 5800 50  0001 C CNN
+F 2 "Pin_Headers:Pin_Header_Angled_1x02_Pitch2.54mm" H 9900 5800 50  0001 C CNN
 F 3 "" H 9900 5800 50  0001 C CNN
 	1    9900 5800

Commit message: updated
Parts:
- removed J1: Conn_01x02, Pin_Headers:Pin_Header_Straight_1x02_Pitch2.54mm, symbol Conn_01x02
- removed R17, R18, R2, R4: R, Resistors_SMD:R_0805, symbol R
- added JP3, JP4: Jumper_NO_Small, Pin_Headers:Pin_Header_Angled_1x02_Pitch2.54mm, symbol Jumper_NO_Small
- U5: footprint Housings_SSOP:VSSOP-8_2.3x2mm_Pitch0.5mm -> Housings_SSOP:SSOP-8_2.95x2.8mm_Pitch0.65mm
Connections:
- net labels added: SCL_HI, SCL_LO, SDA_HI, SDA_LO
- net labels removed: +5V, -5V, GNDREF, SCL, SDA, VREF1
- wire segments 173 -> 170
- no-connect marks 29 -> 33
Other:
- moved on the sheet: U2C, U2D

Commit message: pcb opamps v1
Parts:
- removed C15, C16: C, Capacitors_SMD:C_0805, symbol C
- removed JP2: Jumper_NO_Small, Pin_Headers:Pin_Header_Angled_1x02_Pitch2.54mm, symbol Jumper_NO_Small
- J7: renamed from J8; footprint Connectors_Molex:Molex_MiniFit-JR-5569-04A2_2x02x4.20mm_Angled -> Pin_Headers:Pin_Header_Straight_1x04_Pitch2.54mm
- JP1: footprint Pin_Headers:Pin_Header_Angled_1x02_Pitch2.54mm -> Pin_Headers:Pin_Header_Straight_1x02_Pitch2.54mm
- JP2: renamed from JP3; footprint Pin_Headers:Pin_Header_Angled_1x02_Pitch2.54mm -> Pin_Headers:Pin_Header_Straight_1x02_Pitch2.54mm
- JP3: renamed from JP4; footprint Pin_Headers:Pin_Header_Angled_1x02_Pitch2.54mm -> Pin_Headers:Pin_Header_Straight_1x02_Pitch2.54mm
- renumbered C9 to C10, C10 to C11, C11 to C12, C12 to C13, C13 to C14, C14 to C15, C24 to C18, C17 to C19, C18 to C20, C19 to C21, C20 to C22, C21 to C23, C22 to C24, C27 to C25, C25 to C26, C26 to C27, C23 to C9, J2 to J1, J3 to J2, J4 to J3, J6 to J4, J7 to J6, R11 to R10, R12 to R11, R13 to R12, R14 to R13, R15 to R14, R21 to R15, R22 to R16, R23 to R17, R24 to R18, R25 to R19, R3 to R2, R19 to R20, R20 to R21, R5 to R3, R6 to R4, R16 to R5, R7 to R6, R8 to R7, R9 to R8, R10 to R9, U5 to U4, U4 to U5
Connections:
- net labels removed: 3V3, 5V, VCC_OPAMP, V_DPU, Vcc
- wire segments 170 -> 166

Commit message: pcb v1
Connections:
- net labels removed: Earth
Changed lines of the file:
@@
-$EndComp
-$Comp
-L Earth #PWR01
-U 1 1 5A3AB17D
-P 6300 4000
-F 0 "#PWR01" H 6300 3750 50  0001 C CNN
-F 1 "Earth" H 6300 3850 50  0001 C CNN
-F 2 "" H 6300 4000 50  0001 C CNN
-F 3 "" H 6300 4000 50  0001 C CNN
-	1    6300 4000
-	1    0    0    -1
 $EndComp
 $Comp
@@
 F 3 "" H 5000 2900 50  0001 C CNN
 	1    5000 2900
-	1    0    0    -1
-$EndComp
-$Comp
-L Earth #PWR02
-U 1 1 5A3AB279
-P 5150 2850
-F 0 "#PWR02" H 5150 2600 50  0001 C CNN
-F 1 "Earth" H 5150 2700 50  0001 C CNN
-F 2 "" H 5150 2850 50  0001 C CNN
-F 3 "" H 5150 2850 50  0001 C CNN
-	1    5150 2850
 	1    0    0    -1
 $EndComp
@@
 $EndComp
 $Comp
-L Earth #PWR03
-U 1 1 5A3C6AC1
-P 3600 2700
-F 0 "#PWR03" H 3600 2450 50  0001 C CNN
-F 1 "Earth" H 3600 2550 50  0001 C CNN
-F 2 "" H 3600 2700 50  0001 C CNN
-F 3 "" H 3600 2700 50  0001 C CNN
-	1    3600 2700
-	1    0    0    -1
-$EndComp
-$Comp
 L C C1
 U 1 1 5A3C7A68
@@
 $EndComp
 $Comp
-L Earth #PWR04
-U 1 1 5A3C7C72
-P 1400 3000
-F 0 "#PWR04" H 1400 2750 50  0001 C CNN
-F 1 "Earth" H 1400 2850 50  0001 C CNN
-F 2 "" H 1400 3000 50  0001 C CNN
-F 3 "" H 1400 3000 50  0001 C CNN
-	1    1400 3000
-	1    0    0    -1
-$EndComp
-$Comp
-L Earth #PWR05
-U 1 1 5A3C7CA8
-P 1100 3000
-F 0 "#PWR05" H 1100 2750 50  0001 C CNN
-F 1 "Earth" H 1100 2850 50  0001 C CNN
-F 2 "" H 1100 3000 50  0001 C CNN
-F 3 "" H 1100 3000 50  0001 C CNN
-	1    1100 3000
-	1    0    0    -1
-$EndComp
-$Comp
 L R R1
 U 1 1 5A3C7DB9
@@
 $EndComp
 $Comp
-L Earth #PWR06
-U 1 1 5A3C7ED5
-P 1600 3200
-F 0 "#PWR06" H 1600 2950 50  0001 C CNN
-F 1 "Earth" H 1600 3050 50  0001 C CNN
-F 2 "" H 1600 3200 50  0001 C CNN
-F 3 "" H 1600 3200 50  0001 C CNN
-	1    1600 3200
-	1    0    0    -1
-$EndComp
-$Comp
 L R R2
 U 1 1 5A3C80F5
@@
 $EndComp
 $Comp
-L Earth #PWR07
-U 1 1 5A3C9145
-P 2450 3150
-F 0 "#PWR07" H 2450 2900 50  0001 C CNN
-F 1 "Earth" H 2450 3000 50  0001 C CNN
-F 2 "" H 2450 3150 50  0001 C CNN
-F 3 "" H 2450 3150 50  0001 C CNN
-	1    2450 3150
-	1    0    0    -1
-$EndComp
-$Comp
 L R R6
 U 1 1 5A3C959E
@@
 $EndComp
 $Comp
-L Earth #PWR08
-U 1 1 5A3CA1FF
-P 4600 2800
-F 0 "#PWR08" H 4600 2550 50  0001 C CNN
-F 1 "Earth" H 4600 2650 50  0001 C CNN
-F 2 "" H 4600 2800 50  0001 C CNN
-F 3 "" H 4600 2800 50  0001 C CNN
-	1    4600 2800
-	1    0    0    -1
-$EndComp
-$Comp
 L C C21
 U 1 1 5A3CB9C9
@@
 $EndComp
 $Comp
-L Earth #PWR09
-U 1 1 5A3CFC85
-P 5700 2800
-F 0 "#PWR09" H 5700 2550 50  0001 C CNN
-F 1 "Earth" H 5700 2650 50  0001 C CNN
-F 2 "" H 5700 2800 50  0001 C CNN
-F 3 "" H 5700 2800 50  0001 C CNN
-	1    5700 2800
-	1    0    0    -1
-$EndComp
-$Comp
 L C C24
 U 1 1 5A3D039C
@@
 $EndComp
 $Comp
-L Earth #PWR010
-U 1 1 5A3D1F4E
-P 6900 4400
-F 0 "#PWR010" H 6900 4150 50  0001 C CNN
-F 1 "Earth" H 6900 4250 50  0001 C CNN
-F 2 "" H 6900 4400 50  0001 C CNN
-F 3 "" H 6900 4400 50  0001 C CNN
-	1    6900 4400
-	1    0    0    -1
-$EndComp
-$Comp
 L C C13
 U 1 1 5A3D48EC
@@
 $EndComp
 $Comp
-L Earth #PWR011
-U 1 1 5A3D4E8F
-P 4200 3000
-F 0 "#PWR011" H 4200 2750 50  0001 C CNN
-F 1 "Earth" H 4200 2850 50  0001 C CNN
-F 2 "" H 4200 3000 50  0001 C CNN
-F 3 "" H 4200 3000 50  0001 C CNN
-	1    4200 3000
-	1    0    0    -1
-$EndComp
-$Comp
-L Earth #PWR012
-U 1 1 5A3D4EE5
-P 4200 3600
-F 0 "#PWR012" H 4200 3350 50  0001 C CNN
-F 1 "Earth" H 4200 3450 50  0001 C CNN
-F 2 "" H 4200 3600 50  0001 C CNN
-F 3 "" H 4200 3600 50  0001 C CNN
-	1    4200 3600
-	1    0    0    -1
-$EndComp
-$Comp
 L C C11
 U 1 1 5A3D4F3B
@@
 	1    4000 5900
 	0    1    1    0
-$EndComp
-$Comp
-L Earth #PWR013
-U 1 1 5A3DE714
-P 5700 5900
-F 0 "#PWR013" H 5700 5650 50  0001 C CNN
-F 1 "Earth" H 5700 5750 50  0001 C CNN
-F 2 "" H 5700 5900 50  0001 C CNN
-F 3 "" H 5700 5900 50  0001 C CNN
-	1    5700 5900
-	1    0    0    -1
-$EndComp
-$Comp
-L Earth #PWR014
-U 1 1 5A3DE77E
-P 6300 5900
-F 0 "#PWR014" H 6300 5650 50  0001 C CNN
-F 1 "Earth" H 6300 5750 50  0001 C CNN
-F 2 "" H 6300 5900 50  0001 C CNN
-F 3 "" H 6300 5900 50  0001 C CNN
-	1    6300 5900
-	1    0    0    -1
-$EndComp
-$Comp
-L Earth #PWR015
-U 1 1 5A3DE869
-P 5100 5900
-F 0 "#PWR015" H 5100 5650 50  0001 C CNN
-F 1 "Earth" H 5100 5750 50  0001 C CNN
-F 2 "" H 5100 5900 50  0001 C CNN
-F 3 "" H 5100 5900 50  0001 C CNN
-	1    5100 5900
-	1    0    0    -1
 $EndComp
 $Comp
@@
 Wire Wire Line
 	1950 2700 1950 2950
-$Comp
-L Earth #PWR016
-U 1 1 5A4CAFAD
-P 1950 3500
-F 0 "#PWR016" H 1950 3250 50  0001 C CNN
-F 1 "Earth" H 1950 3350 50  0001 C CNN
-F 2 "" H 1950 3500 50  0001 C CNN
-F 3 "" H 1950 3500 50  0001 C CNN
-	1    1950 3500
-	1    0    0    -1
-$EndComp
 Wire Wire Line
 	1950 3500 1950 3250
@@
 	0    1    1    0
 $EndComp
-$Comp
-L Earth #PWR017
-U 1 1 5A4CD3D5
-P 4300 1100
-F 0 "#PWR017" H 4300 850 50  0001 C CNN
-F 1 "Earth" H 4300 950 50  0001 C CNN
-F 2 "" H 4300 1100 50  0001 C CNN
-F 3 "" H 4300 1100 50  0001 C CNN
-	1    4300 1100
-	1    0    0    -1
-$EndComp
 Connection ~ 4900 2200
 Wire Wire Line
@@
 F 3 "" H 3450 2250 50  0001 C CNN
 	1    3450 2250
-	1    0    0    -1
-$EndComp
-$Comp
-L Earth #PWR018
-U 1 1 5A4C3A11
-P 3450 2500
-F 0 "#PWR018" H 3450 2250 50  0001 C CNN
-F 1 "Earth" H 3450 2350 50  0001 C CNN
-F 2 "" H 3450 2500 50  0001 C CNN
-F 3 "" H 3450 2500 50  0001 C CNN
-	1    3450 2500
 	1    0    0    -1
 $EndComp
@@
 Text Label 6150 1450 0    60   ~ 0
 +Vcc
+Text Label 6900 4400 0    60   ~ 0
+GND
+$Comp
+L GND #PWR?
+U 1 1 5AA0DDE2
+P 1100 3000
+F 0 "#PWR?" H 1100 2750 50  0001 C CNN
+F 1 "GND" H 1100 2850 50  0000 C CNN
+F 2 "" H 1100 3000 50  0001 C CNN
+F 3 "" H 1100 3000 50  0001 C CNN
+	1    1100 3000
+	1    0    0    -1
+$EndComp
+$Comp
+L GND #PWR?
+U 1 1 5AA0DEBD
+P 1400 3000
+F 0 "#PWR?" H 1400 2750 50  0001 C CNN
+F 1 "GND" H 1400 2850 50  0000 C CNN
+F 2 "" H 1400 3000 50  0001 C CNN
+F 3 "" H 1400 3000 50  0001 C CNN
+	1    1400 3000
+	1    0    0    -1
+$EndComp
+$Comp
+L GND #PWR?
+U 1 1 5AA0DF98
+P 1600 3200
+F 0 "#PWR?" H 1600 2950 50  0001 C CNN
+F 1 "GND" H 1600 3050 50  0000 C CNN
+F 2 "" H 1600 3200 50  0001 C CNN
+F 3 "" H 1600 3200 50  0001 C CNN
+	1    1600 3200
+	1    0    0    -1
+$EndComp
+$Comp
+L GND #PWR?
+U 1 1 5AA0E073
+P 1950 3500
+F 0 "#PWR?" H 1950 3250 50  0001 C CNN
+F 1 "GND" H 1950 3350 50  0000 C CNN
+F 2 "" H 1950 3500 50  0001 C CNN
+F 3 "" H 1950 3500 50  0001 C CNN
+	1    1950 3500
+	1    0    0    -1
+$EndComp
+$Comp
+L GND #PWR?
+U 1 1 5AA0E14E
+P 2450 3150
+F 0 "#PWR?" H 2450 2900 50  0001 C CNN
+F 1 "GND" H 2450 3000 50  0000 C CNN
+F 2 "" H 2450 3150 50  0001 C CNN
+F 3 "" H 2450 3150 50  0001 C CNN
+	1    2450 3150
+	1    0    0    -1
+$EndComp
+$Comp
+L GND #PWR?
+U 1 1 5AA0E229
+P 3450 2500
+F 0 "#PWR?" H 3450 2250 50  0001 C CNN
+F 1 "GND" H 3450 2350 50  0000 C CNN
+F 2 "" H 3450 2500 50  0001 C CNN
+F 3 "" H 3450 2500 50  0001 C CNN
+	1    3450 2500
+	1    0    0    -1
+$EndComp
+$Comp
+L GND #PWR?
+U 1 1 5AA0E304
+P 3600 2700
+F 0 "#PWR?" H 3600 2450 50  0001 C CNN
+F 1 "GND" H 3600 2550 50  0000 C CNN
+F 2 "" H 3600 2700 50  0001 C CNN
+F 3 "" H 3600 2700 50  0001 C CNN
+	1    3600 2700
+	1    0    0    -1
+$EndComp
+$Comp
+L GND #PWR?
+U 1 1 5AA0E3DF
+P 4300 1100
+F 0 "#PWR?" H 4300 850 50  0001 C CNN
+F 1 "GND" H 4300 950 50  0000 C CNN
+F 2 "" H 4300 1100 50  0001 C CNN
+F 3 "" H 4300 1100 50  0001 C CNN
+	1    4300 1100
+	1    0    0    -1
+$EndComp
+$Comp
+L GND #PWR?
+U 1 1 5AA0F78C
+P 5700 2800
+F 0 "#PWR?" H 5700 2550 50  0001 C CNN
+F 1 "GND" H 5700 2650 50  0000 C CNN
+F 2 "" H 5700 2800 50  0001 C CNN
+F 3 "" H 5700 2800 50  0001 C CNN
+	1    5700 2800
+	1    0    0    -1
+$EndComp
+$Comp
+L GND #PWR?
+U 1 1 5AA0F867
+P 5150 2850
+F 0 "#PWR?" H 5150 2600 50  0001 C CNN
+F 1 "GND" H 5150 2700 50  0000 C CNN
+F 2 "" H 5150 2850 50  0001 C CNN
+F 3 "" H 5150 2850 50  0001 C CNN
+	1    5150 2850
+	1    0    0    -1
+$EndComp
+$Comp
+L GND #PWR?
+U 1 1 5AA0F942
+P 4600 2800
+F 0 "#PWR?" H 4600 2550 50  0001 C CNN
+F 1 "GND" H 4600 2650 50  0000 C CNN
+F 2 "" H 4600 2800 50  0001 C CNN
+F 3 "" H 4600 2800 50  0001 C CNN
+	1    4600 2800
+	1    0    0    -1
+$EndComp
+$Comp
+L GND #PWR?
+U 1 1 5AA0FA1D
+P 4200 3000
+F 0 "#PWR?" H 4200 2750 50  0001 C CNN
+F 1 "GND" H 4200 2850 50  0000 C CNN
+F 2 "" H 4200 3000 50  0001 C CNN
+F 3 "" H 4200 3000 50  0001 C CNN
+	1    4200 3000
+	1    0    0    -1
+$EndComp
+$Comp
+L GND #PWR?
+U 1 1 5AA0FAF8
+P 4200 3600
+F 0 "#PWR?" H 4200 3350 50  0001 C CNN
+F 1 "GND" H 4200 3450 50  0000 C CNN
+F 2 "" H 4200 3600 50  0001 C CNN
+F 3 "" H 4200 3600 50  0001 C CNN
+	1    4200 3600
+	1    0    0    -1
+$EndComp
+$Comp
+L GND #PWR?
+U 1 1 5AA10F29
+P 6300 4000
+F 0 "#PWR?" H 6300 3750 50  0001 C CNN
+F 1 "GND" H 6300 3850 50  0000 C CNN
+F 2 "" H 6300 4000 50  0001 C CNN
+F 3 "" H 6300 4000 50  0001 C CNN
+	1    6300 4000
+	1    0    0    -1
+$EndComp
+$Comp
+L GND #PWR?
+U 1 1 5AA11004
+P 6900 4400
+F 0 "#PWR?" H 6900 4150 50  0001 C CNN
+F 1 "GND" H 6900 4250 50  0000 C CNN
+F 2 "" H 6900 4400 50  0001 C CNN
+F 3 "" H 6900 4400 50  0001 C CNN
+	1    6900 4400
+	1    0    0    -1
+$EndComp
+$Comp
+L GND #PWR?
+U 1 1 5AA181CD
+P 6300 5900
+F 0 "#PWR?" H 6300 5650 50  0001 C CNN
+F 1 "GND" H 6300 5750 50  0000 C CNN
+F 2 "" H 6300 5900 50  0001 C CNN
+F 3 "" H 6300 5900 50  0001 C CNN
+	1    6300 5900
+	1    0    0    -1
+$EndComp
+$Comp
+L GND #PWR?
+U 1 1 5AA18265
+P 5700 5900
+F 0 "#PWR?" H 5700 5650 50  0001 C CNN
+F 1 "GND" H 5700 5750 50  0000 C CNN
+F 2 "" H 5700 5900 50  0001 C CNN
+F 3 "" H 5700 5900 50  0001 C CNN
+	1    5700 5900
+	1    0    0    -1
+$EndComp
+$Comp
+L GND #PWR?
+U 1 1 5AA182FD
+P 5100 5900
+F 0 "#PWR?" H 5100 5650 50  0001 C CNN
+F 1 "GND" H 5100 5750 50  0000 C CNN
+F 2 "" H 5100 5900 50  0001 C CNN
+F 3 "" H 5100 5900 50  0001 C CNN
+	1    5100 5900
+	1    0    0    -1
+$EndComp
 $EndSCHEMATC
