File: variable_load.sch (KiCad schematic (older format))
At the start: 63 parts, among them J1 Conn_01x04, J2 LEMO, J3 Conn_01x02, J4 GS3, J5 Conn_01x04, J6 Conn_01x04, J7 Conn_01x04, Q1 NTD4858N, U1 DAC5578, U2 LM324, U3 TLV1117-33, U4 PCA9306, U5 adafruit_ft232h, U6 APD123

Commit message: pcb v2
Parts:
- added D1: LED, LEDs:LED_1206_HandSoldering, symbol LED
- added R22: R, Resistors_SMD:R_0805, symbol R
Connections:
- wire segments 166 -> 169
Changed lines of the file:
@@
 $EndComp
 $Comp
-L GND #PWR019
+L GND #PWR01
 U 1 1 5A668DEC
 P 10550 1750
-F 0 "#PWR019" H 10550 1500 50  0001 C CNN
+F 0 "#PWR01" H 10550 1500 50  0001 C CNN
 F 1 "GND" H 10550 1600 50  0000 C CNN
 F 2 "" H 10550 1750 50  0001 C CNN
@@
 $EndComp
 $Comp
-L GND #PWR020
+L GND #PWR02
 U 1 1 5A668E7A
 P 10800 1750
-F 0 "#PWR020" H 10800 1500 50  0001 C CNN
+F 0 "#PWR02" H 10800 1500 50  0001 C CNN
 F 1 "GND" H 10800 1600 50  0000 C CNN
 F 2 "" H 10800 1750 50  0001 C CNN
@@
 $EndComp
 $Comp
-L GND #PWR021
+L GND #PWR03
 U 1 1 5A66AD0F
 P 9300 1750
-F 0 "#PWR021" H 9300 1500 50  0001 C CNN
+F 0 "#PWR03" H 9300 1500 50  0001 C CNN
 F 1 "GND" H 9300 1600 50  0000 C CNN
 F 2 "" H 9300 1750 50  0001 C CNN
@@
 $EndComp
 $Comp
-L GND #PWR022
+L GND #PWR04
 U 1 1 5A66AD9F
 P 9900 1750
-F 0 "#PWR022" H 9900 1500 50  0001 C CNN
+F 0 "#PWR04" H 9900 1500 50  0001 C CNN
 F 1 "GND" H 9900 1600 50  0000 C CNN
 F 2 "" H 9900 1750 50  0001 C CNN
@@
 $EndComp
 $Comp
-L GND #PWR023
+L GND #PWR05
 U 1 1 5A66CD96
 P 8600 4600
-F 0 "#PWR023" H 8600 4350 50  0001 C CNN
+F 0 "#PWR05" H 8600 4350 50  0001 C CNN
 F 1 "GND" H 8600 4450 50  0000 C CNN
 F 2 "" H 8600 4600 50  0001 C CNN
@@
 SDA_HI
 $Comp
-L GND #PWR024
+L GND #PWR06
 U 1 1 5A67066D
 P 10050 2900
-F 0 "#PWR024" H 10050 2650 50  0001 C CNN
+F 0 "#PWR06" H 10050 2650 50  0001 C CNN
 F 1 "GND" H 10050 2750 50  0000 C CNN
 F 2 "" H 10050 2900 50  0001 C CNN
@@
 Connection ~ 10600 3800
 $Comp
-L PWR_FLAG #FLG025
+L PWR_FLAG #FLG07
 U 1 1 5A685722
 P 10600 4500
-F 0 "#FLG025" H 10600 4575 50  0001 C CNN
+F 0 "#FLG07" H 10600 4575 50  0001 C CNN
 F 1 "PWR_FLAG" H 10600 4650 50  0000 C CNN
 F 2 "" H 10600 4500 50  0001 C CNN
@@
 $EndComp
 $Comp
-L GND #PWR026
+L GND #PWR08
 U 1 1 5A6859AC
 P 10600 4800
-F 0 "#PWR026" H 10600 4550 50  0001 C CNN
+F 0 "#PWR08" H 10600 4550 50  0001 C CNN
 F 1 "GND" H 10600 4650 50  0000 C CNN
 F 2 "" H 10600 4800 50  0001 C CNN
@@
 $EndComp
 $Comp
-L GND #PWR027
+L GND #PWR09
 U 1 1 5A68B41A
 P 8850 5050
-F 0 "#PWR027" H 8850 4800 50  0001 C CNN
+F 0 "#PWR09" H 8850 4800 50  0001 C CNN
 F 1 "GND" H 8850 4900 50  0000 C CNN
 F 2 "" H 8850 5050 50  0001 C CNN
@@
 	4900 2000 4500 2000
 $Comp
-L GND #PWR028
+L GND #PWR010
 U 1 1 5A710C83
 P 8350 6250
-F 0 "#PWR028" H 8350 6000 50  0001 C CNN
+F 0 "#PWR010" H 8350 6000 50  0001 C CNN
 F 1 "GND" H 8350 6100 50  0000 C CNN
 F 2 "" H 8350 6250 50  0001 C CNN
@@
 $EndComp
 $Comp
-L GND #PWR029
+L GND #PWR011
 U 1 1 5A715B55
 P 10600 4000
-F 0 "#PWR029" H 10600 3750 50  0001 C CNN
+F 0 "#PWR011" H 10600 3750 50  0001 C CNN
 F 1 "GND" H 10600 3850 50  0000 C CNN
 F 2 "" H 10600 4000 50  0001 C CNN
@@
 $EndComp
 $Comp
-L GND #PWR030
+L GND #PWR012
 U 1 1 5A718759
 P 3100 1600
-F 0 "#PWR030" H 3100 1350 50  0001 C CNN
+F 0 "#PWR012" H 3100 1350 50  0001 C CNN
 F 1 "GND" H 3100 1450 50  0000 C CNN
 F 2 "" H 3100 1600 50  0001 C CNN
@@
 +Vcc
 $Comp
-L PWR_FLAG #FLG031
+L PWR_FLAG #FLG013
 U 1 1 5A732DC7
 P 4350 5200
-F 0 "#FLG031" H 4350 5275 50  0001 C CNN
+F 0 "#FLG013" H 4350 5275 50  0001 C CNN
 F 1 "PWR_FLAG" H 4350 5350 50  0000 C CNN
 F 2 "" H 4350 5200 50  0001 C CNN
@@
 $EndComp
 $Comp
-L PWR_FLAG #FLG032
+L PWR_FLAG #FLG014
 U 1 1 5A732E61
 P 2000 5900
-F 0 "#FLG032" H 2000 5975 50  0001 C CNN
+F 0 "#FLG014" H 2000 5975 50  0001 C CNN
 F 1 "PWR_FLAG" H 2000 6050 50  0000 C CNN
 F 2 "" H 2000 5900 50  0001 C CNN
@@
 $EndComp
 $Comp
-L PWR_FLAG #FLG033
+L PWR_FLAG #FLG015
 U 1 1 5A732F81
 P 2700 5900
-F 0 "#FLG033" H 2700 5975 50  0001 C CNN
+F 0 "#FLG015" H 2700 5975 50  0001 C CNN
 F 1 "PWR_FLAG" H 2700 6050 50  0000 C CNN
 F 2 "" H 2700 5900 50  0001 C CNN
@@
 $EndComp
 $Comp
-L GND #PWR034
+L GND #PWR016
 U 1 1 5A73D415
 P 5700 1450
-F 0 "#PWR034" H 5700 1200 50  0001 C CNN
+F 0 "#PWR016" H 5700 1200 50  0001 C CNN
 F 1 "GND" H 5700 1300 50  0000 C CNN
 F 2 "" H 5700 1450 50  0001 C CNN
@@
 GND
 $Comp
-L GND #PWR?
+L GND #PWR017
 U 1 1 5AA0DDE2
 P 1100 3000
-F 0 "#PWR?" H 1100 2750 50  0001 C CNN
+F 0 "#PWR017" H 1100 2750 50  0001 C CNN
 F 1 "GND" H 1100 2850 50  0000 C CNN
 F 2 "" H 1100 3000 50  0001 C CNN
@@
 $EndComp
 $Comp
-L GND #PWR?
+L GND #PWR018
 U 1 1 5AA0DEBD
 P 1400 3000
-F 0 "#PWR?" H 1400 2750 50  0001 C CNN
+F 0 "#PWR018" H 1400 2750 50  0001 C CNN
 F 1 "GND" H 1400 2850 50  0000 C CNN
 F 2 "" H 1400 3000 50  0001 C CNN
@@
 $EndComp
 $Comp
-L GND #PWR?
+L GND #PWR019
 U 1 1 5AA0DF98
 P 1600 3200
-F 0 "#PWR?" H 1600 2950 50  0001 C CNN
+F 0 "#PWR019" H 1600 2950 50  0001 C CNN
 F 1 "GND" H 1600 3050 50  0000 C CNN
 F 2 "" H 1600 3200 50  0001 C CNN
@@
 $EndComp
 $Comp
-L GND #PWR?
+L GND #PWR020
 U 1 1 5AA0E073
 P 1950 3500
-F 0 "#PWR?" H 1950 3250 50  0001 C CNN
+F 0 "#PWR020" H 1950 3250 50  0001 C CNN
 F 1 "GND" H 1950 3350 50  0000 C CNN
 F 2 "" H 1950 3500 50  0001 C CNN
@@
 $EndComp
 $Comp
-L GND #PWR?
+L GND #PWR021
 U 1 1 5AA0E14E
 P 2450 3150
-F 0 "#PWR?" H 2450 2900 50  0001 C CNN
+F 0 "#PWR021" H 2450 2900 50  0001 C CNN
 F 1 "GND" H 2450 3000 50  0000 C CNN
 F 2 "" H 2450 3150 50  0001 C CNN
@@
 $EndComp
 $Comp
-L GND #PWR?
+L GND #PWR022
 U 1 1 5AA0E229
 P 3450 2500
-F 0 "#PWR?" H 3450 2250 50  0001 C CNN
+F 0 "#PWR022" H 3450 2250 50  0001 C CNN
 F 1 "GND" H 3450 2350 50  0000 C CNN
 F 2 "" H 3450 2500 50  0001 C CNN
@@
 $EndComp
 $Comp
-L GND #PWR?
+L GND #PWR023
 U 1 1 5AA0E304
 P 3600 2700
-F 0 "#PWR?" H 3600 2450 50  0001 C CNN
+F 0 "#PWR023" H 3600 2450 50  0001 C CNN
 F 1 "GND" H 3600 2550 50  0000 C CNN
 F 2 "" H 3600 2700 50  0001 C CNN
@@
 $EndComp
 $Comp
-L GND #PWR?
+L GND #PWR024
 U 1 1 5AA0E3DF
 P 4300 1100
-F 0 "#PWR?" H 4300 850 50  0001 C CNN
+F 0 "#PWR024" H 4300 850 50  0001 C CNN
 F 1 "GND" H 4300 950 50  0000 C CNN
 F 2 "" H 4300 1100 50  0001 C CNN
@@
 $EndComp
 $Comp
-L GND #PWR?
+L GND #PWR025
 U 1 1 5AA0F78C
 P 5700 2800
-F 0 "#PWR?" H 5700 2550 50  0001 C CNN
+F 0 "#PWR025" H 5700 2550 50  0001 C CNN
 F 1 "GND" H 5700 2650 50  0000 C CNN
 F 2 "" H 5700 2800 50  0001 C CNN
@@
 $EndComp
 $Comp
-L GND #PWR?
+L GND #PWR026
 U 1 1 5AA0F867
 P 5150 2850
-F 0 "#PWR?" H 5150 2600 50  0001 C CNN
+F 0 "#PWR026" H 5150 2600 50  0001 C CNN
 F 1 "GND" H 5150 2700 50  0000 C CNN
 F 2 "" H 5150 2850 50  0001 C CNN
@@
 $EndComp
 $Comp
-L GND #PWR?
+L GND #PWR027
 U 1 1 5AA0F942
 P 4600 2800
-F 0 "#PWR?" H 4600 2550 50  0001 C CNN
+F 0 "#PWR027" H 4600 2550 50  0001 C CNN
 F 1 "GND" H 4600 2650 50  0000 C CNN
 F 2 "" H 4600 2800 50  0001 C CNN
@@
 $EndComp
 $Comp
-L GND #PWR?
+L GND #PWR028
 U 1 1 5AA0FA1D
 P 4200 3000
-F 0 "#PWR?" H 4200 2750 50  0001 C CNN
+F 0 "#PWR028" H 4200 2750 50  0001 C CNN
 F 1 "GND" H 4200 2850 50  0000 C CNN
 F 2 "" H 4200 3000 50  0001 C CNN
@@
 $EndComp
 $Comp
-L GND #PWR?
+L GND #PWR029
 U 1 1 5AA0FAF8
 P 4200 3600
-F 0 "#PWR?" H 4200 3350 50  0001 C CNN
+F 0 "#PWR029" H 4200 3350 50  0001 C CNN
 F 1 "GND" H 4200 3450 50  0000 C CNN
 F 2 "" H 4200 3600 50  0001 C CNN
@@
 $EndComp
 $Comp
-L GND #PWR?
+L GND #PWR030
 U 1 1 5AA10F29
 P 6300 4000
-F 0 "#PWR?" H 6300 3750 50  0001 C CNN
+F 0 "#PWR030" H 6300 3750 50  0001 C CNN
 F 1 "GND" H 6300 3850 50  0000 C CNN
 F 2 "" H 6300 4000 50  0001 C CNN
@@
 $EndComp
 $Comp
-L GND #PWR?
+L GND #PWR031
 U 1 1 5AA11004
 P 6900 4400
-F 0 "#PWR?" H 6900 4150 50  0001 C CNN
+F 0 "#PWR031" H 6900 4150 50  0001 C CNN
 F 1 "GND" H 6900 4250 50  0000 C CNN
 F 2 "" H 6900 4400 50  0001 C CNN
@@
 $EndComp
 $Comp
-L GND #PWR?
+L GND #PWR032
 U 1 1 5AA181CD
 P 6300 5900
-F 0 "#PWR?" H 6300 5650 50  0001 C CNN
+F 0 "#PWR032" H 6300 5650 50  0001 C CNN
 F 1 "GND" H 6300 5750 50  0000 C CNN
 F 2 "" H 6300 5900 50  0001 C CNN
@@
 $EndComp
 $Comp
-L GND #PWR?
+L GND #PWR033
 U 1 1 5AA18265
 P 5700 5900
-F 0 "#PWR?" H 5700 5650 50  0001 C CNN
+F 0 "#PWR033" H 5700 5650 50  0001 C CNN
 F 1 "GND" H 5700 5750 50  0000 C CNN
 F 2 "" H 5700 5900 50  0001 C CNN
@@
 $EndComp
 $Comp
-L GND #PWR?
+L GND #PWR034
 U 1 1 5AA182FD
 P 5100 5900
-F 0 "#PWR?" H 5100 5650 50  0001 C CNN
+F 0 "#PWR034" H 5100 5650 50  0001 C CNN
 F 1 "GND" H 5100 5750 50  0000 C CNN
 F 2 "" H 5100 5900 50  0001 C CNN
@@
 	1    0    0    -1
 $EndComp
+$Comp
+L LED D1
+U 1 1 5AA8442E
+P 4750 6500
+F 0 "D1" H 4750 6600 50  0000 C CNN
+F 1 "LED" H 4750 6400 50  0000 C CNN
+F 2 "LEDs:LED_1206_HandSoldering" H 4750 6500 50  0001 C CNN
+F 3 "" H 4750 6500 50  0001 C CNN
+	1    4750 6500
+	1    0    0    -1
+$EndComp
+$Comp
+L R R22
+U 1 1 5AA8AAE3
+P 5250 6500
+F 0 "R22" V 5330 6500 50  0000 C CNN
+F 1 "R" V 5250 6500 50  0000 C CNN
+F 2 "Resistors_SMD:R_0805" V 5180 6500 50  0001 C CNN
+F 3 "" H 5250 6500 50  0001 C CNN
+	1    5250 6500
+	0    1    1    0
+$EndComp
+Wire Wire Line
+	4900 6500 5100 6500
+Wire Wire Line
+	5400 6500 5600 6500
+Wire Wire Line
+	4600 6500 4450 6500
+$Comp
+L GND #PWR035
+U 1 1 5AA8B472
+P 4450 6500
+F 0 "#PWR035" H 4450 6250 50  0001 C CNN
+F 1 "GND" H 4450 6350 50  0000 C CNN
+F 2 "" H 4450 6500 50  0001 C CNN
+F 3 "" H 4450 6500 50  0001 C CNN
+	1    4450 6500
+	1    0    0    -1
+$EndComp
+Text Label 5600 6500 0    60   ~ 0
++Vcc
 $EndSCHEMATC
