File: variable_load.sch (KiCad schematic (older format))
At the start: 65 parts, among them J1 Conn_01x04, J2 LEMO, J3 Conn_01x02, J4 GS3, J5 Conn_01x04, J6 Conn_01x04, J7 Conn_01x04, Q1 NTD4858N, U1 DAC5578, U2 LM324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

Commit message: pcb v3
Parts:
- added J8, J9: Conn_01x02, Pin_Headers:Pin_Header_Straight_1x02_Pitch2.54mm, symbol Conn_01x02
Connections:
- wire segments 169 -> 177
Other:
- moved on the sheet: C5, C6
Changed lines of the file:
@@
 Connection ~ 7400 2300
 Wire Wire Line
-	7400 2300 7400 2400
-Wire Wire Line
-	7400 2600 7400 2500
+	7400 2150 7400 2400
+Wire Wire Line
+	7400 2500 7400 2750
 Wire Wire Line
 	5000 4100 4600 4100
@@
 Wire Wire Line
 	4600 3600 4700 3600
-Connection ~ 2300 5600
-Connection ~ 3000 5600
-Connection ~ 3000 5300
+Connection ~ 2800 5300
+Connection ~ 2800 5000
 Connection ~ 1600 5300
 Connection ~ 1600 5600
-Wire Wire Line
-	2300 5000 2300 6000
-Connection ~ 2300 5300
 $Comp
 L C C6
 U 1 1 5A3DACAD
-P 2650 5600
-F 0 "C6" H 2675 5700 50  0000 L CNN
-F 1 "C" H 2675 5500 50  0000 L CNN
-F 2 "Capacitors_SMD:C_0805" H 2688 5450 50  0001 C CNN
-F 3 "" H 2650 5600 50  0001 C CNN
-	1    2650 5600
+P 2450 5300
+F 0 "C6" H 2475 5400 50  0000 L CNN
+F 1 "C" H 2475 5200 50  0000 L CNN
+F 2 "Capacitors_SMD:C_0805" H 2488 5150 50  0001 C CNN
+F 3 "" H 2450 5300 50  0001 C CNN
+	1    2450 5300
 	0    1    1    0
 $EndComp
@@
 L C C5
 U 1 1 5A3DAD8E
-P 2650 5300
-F 0 "C5" H 2675 5400 50  0000 L CNN
-F 1 "C" H 2675 5200 50  0000 L CNN
-F 2 "Capacitors_SMD:C_0805" H 2688 5150 50  0001 C CNN
-F 3 "" H 2650 5300 50  0001 C CNN
-	1    2650 5300
+P 2450 5000
+F 0 "C5" H 2475 5100 50  0000 L CNN
+F 1 "C" H 2475 4900 50  0000 L CNN
+F 2 "Capacitors_SMD:C_0805" H 2488 4850 50  0001 C CNN
+F 3 "" H 2450 5000 50  0001 C CNN
+	1    2450 5000
 	0    1    1    0
 $EndComp
@@
 $EndComp
 Wire Wire Line
-	3000 5600 2800 5600
-Wire Wire Line
-	2100 5600 2500 5600
-Wire Wire Line
-	2800 5300 3000 5300
-Wire Wire Line
-	2100 5300 2500 5300
+	2800 5300 2600 5300
+Wire Wire Line
+	2600 5000 2800 5000
 Wire Wire Line
 	1600 5300 1800 5300
@@
 Text Label 1600 5000 0    60   ~ 0
 +Vcc
-Text Label 3000 5000 0    60   ~ 0
+Text Label 2800 4700 0    60   ~ 0
 -Vcc
-Text Label 2300 5000 0    60   ~ 0
+Text Label 2700 5900 0    60   ~ 0
 GND
 Text Label 4000 5700 0    60   ~ 0
@@
 Text Label 3900 4800 0    60   ~ 0
 3V3LDO
-Text Label 7700 2350 0    60   ~ 0
+Text Label 7600 2400 0    60   ~ 0
 Vin
-Text Label 7700 2600 0    60   ~ 0
+Text Label 7600 2600 0    60   ~ 0
 Vin_rtn
 Text Label 5100 1100 0    60   ~ 0
@@
 $EndComp
 Wire Wire Line
-	3000 5000 3000 6000
+	2800 5700 2800 4700
 Wire Wire Line
 	1600 5000 1600 6000
 Wire Wire Line
 	1600 6000 2200 6000
-Wire Wire Line
-	3000 6000 2500 6000
-Connection ~ 2400 5600
-Connection ~ 2400 5300
-Wire Wire Line
-	2400 5000 2400 6000
 $Comp
 L R R3
@@
 L PWR_FLAG #FLG015
 U 1 1 5A732F81
-P 2700 5900
-F 0 "#FLG015" H 2700 5975 50  0001 C CNN
-F 1 "PWR_FLAG" H 2700 6050 50  0000 C CNN
-F 2 "" H 2700 5900 50  0001 C CNN
-F 3 "" H 2700 5900 50  0001 C CNN
-	1    2700 5900
-	1    0    0    -1
-$EndComp
-Wire Wire Line
-	2700 6000 2700 5900
-Connection ~ 2700 6000
+P 2500 5600
+F 0 "#FLG015" H 2500 5675 50  0001 C CNN
+F 1 "PWR_FLAG" H 2500 5750 50  0000 C CNN
+F 2 "" H 2500 5600 50  0001 C CNN
+F 3 "" H 2500 5600 50  0001 C CNN
+	1    2500 5600
+	1    0    0    -1
+$EndComp
+Wire Wire Line
+	2500 5700 2500 5600
+Connection ~ 2500 5700
 Wire Wire Line
 	2000 6000 2000 5900
@@
 Text Label 5600 6500 0    60   ~ 0
 +Vcc
+$Comp
+L Conn_01x02 J8
+U 1 1 5AAADB35
+P 4300 1400
+F 0 "J8" H 4300 1500 50  0000 C CNN
+F 1 "Conn_01x02" H 4300 1200 50  0000 C CNN
+F 2 "Pin_Headers:Pin_Header_Straight_1x02_Pitch2.54mm" H 4300 1400 50  0001 C CNN
+F 3 "" H 4300 1400 50  0001 C CNN
+	1    4300 1400
+	1    0    0    -1
+$EndComp
+Wire Wire Line
+	4100 1400 4100 1100
+Connection ~ 4100 1100
+Wire Wire Line
+	3600 1500 4100 1500
+Connection ~ 3600 1500
+$Comp
+L Conn_01x02 J9
+U 1 1 5AAAF82F
+P 8000 2400
+F 0 "J9" H 8000 2500 50  0000 C CNN
+F 1 "Conn_01x02" H 8000 2200 50  0000 C CNN
+F 2 "Pin_Headers:Pin_Header_Straight_1x02_Pitch2.54mm" H 8000 2400 50  0001 C CNN
+F 3 "" H 8000 2400 50  0001 C CNN
+	1    8000 2400
+	1    0    0    -1
+$EndComp
+Wire Wire Line
+	7400 2150 7800 2150
+Wire Wire Line
+	7800 2150 7800 2400
+Wire Wire Line
+	7400 2750 7800 2750
+Wire Wire Line
+	7800 2750 7800 2500
+Wire Wire Line
+	2300 6000 2300 5700
+Wire Wire Line
+	2300 5700 2800 5700
+Wire Wire Line
+	2400 6000 2400 5900
+Wire Wire Line
+	2400 5900 2700 5900
+Wire Wire Line
+	2500 6000 2500 5900
+Connection ~ 2500 5900
+Wire Wire Line
+	2100 5600 2100 5100
+Wire Wire Line
+	2300 5300 2300 4700
+Text Label 2300 4700 0    60   ~ 0
+GND
+Text Label 2100 5100 0    60   ~ 0
+GND
 $EndSCHEMATC

Commit message: pcb v4
Connections:
- wire segments 177 -> 179
Other:
- moved on the sheet: C26
Changed lines of the file:
@@
 Wire Wire Line
 	10050 2900 10050 2700
-Text Label 10150 2500 0    60   ~ 0
+Text Label 10150 2600 0    60   ~ 0
 VREF
-Text Label 10150 2600 0    60   ~ 0
+Text Label 10050 2900 0    60   ~ 0
 SCL_LO
 Text Label 10150 2800 0    60   ~ 0
@@
 L C C26
 U 1 1 5A66AA06
-P 9300 1500
-F 0 "C26" H 9325 1600 50  0000 L CNN
-F 1 "1uF" H 9325 1400 50  0000 L CNN
-F 2 "Capacitors_SMD:C_0805" H 9338 1350 50  0001 C CNN
-F 3 "" H 9300 1500 50  0001 C CNN
-	1    9300 1500
+P 9000 1200
+F 0 "C26" H 9025 1300 50  0000 L CNN
+F 1 "1uF" H 9025 1100 50  0000 L CNN
+F 2 "Capacitors_SMD:C_0805" H 9038 1050 50  0001 C CNN
+F 3 "" H 9000 1200 50  0001 C CNN
+	1    9000 1200
 	1    0    0    -1
 $EndComp
@@
 L GND #PWR03
 U 1 1 5A66AD0F
-P 9300 1750
-F 0 "#PWR03" H 9300 1500 50  0001 C CNN
-F 1 "GND" H 9300 1600 50  0000 C CNN
-F 2 "" H 9300 1750 50  0001 C CNN
-F 3 "" H 9300 1750 50  0001 C CNN
-	1    9300 1750
+P 9000 1450
+F 0 "#PWR03" H 9000 1200 50  0001 C CNN
+F 1 "GND" H 9000 1300 50  0000 C CNN
+F 2 "" H 9000 1450 50  0001 C CNN
+F 3 "" H 9000 1450 50  0001 C CNN
+	1    9000 1450
 	1    0    0    -1
 $EndComp
@@
 L GND #PWR06
 U 1 1 5A67066D
-P 10050 2900
-F 0 "#PWR06" H 10050 2650 50  0001 C CNN
-F 1 "GND" H 10050 2750 50  0000 C CNN
-F 2 "" H 10050 2900 50  0001 C CNN
-F 3 "" H 10050 2900 50  0001 C CNN
-	1    10050 2900
-	1    0    0    -1
+P 10150 2400
+F 0 "#PWR06" H 10150 2150 50  0001 C CNN
+F 1 "GND" H 10150 2250 50  0000 C CNN
+F 2 "" H 10150 2400 50  0001 C CNN
+F 3 "" H 10150 2400 50  0001 C CNN
+	1    10150 2400
+	-1   0    0    1
 $EndComp
 Text Label 10900 900  0    60   ~ 0
 VREF
-Text Label 9150 900  0    60   ~ 0
+Text Label 8750 900  0    60   ~ 0
 +Vcc
 NoConn ~ 9200 2900
@@
 $EndComp
 Wire Wire Line
-	9150 900  9400 900
+	8750 900  9400 900
 Wire Wire Line
 	9400 1200 9300 1200
@@
 	9900 1750 9900 1450
 Wire Wire Line
-	9300 1750 9300 1650
+	9000 1450 9000 1350
 Wire Wire Line
 	9300 1200 9300 1350
@@
 Text Label 2100 5100 0    60   ~ 0
 GND
+Wire Wire Line
+	10150 2500 10150 2400
+Wire Wire Line
+	9000 1050 9000 900
+Connection ~ 9000 900
+Text Label 9300 1350 0    60   ~ 0
++Vcc
 $EndSCHEMATC

Commit message: pcb v5
Parts:
- added C16: C, Capacitors_SMD:C_0805, symbol C
- added J10: Conn_01x02, Pin_Headers:Pin_Header_Straight_1x02_Pitch2.54mm, symbol Conn_01x02
Connections:
- wire segments 179 -> 182
Changed lines of the file:
@@
 Connection ~ 6600 2500
 Wire Wire Line
-	6100 2100 6100 2500
+	6100 2000 6100 2500
 Wire Wire Line
 	6400 2500 6600 2500
@@
 Text Label 9300 1350 0    60   ~ 0
 +Vcc
+$Comp
+L C C16
+U 1 1 5AB9919F
+P 6100 1850
+F 0 "C16" H 6125 1950 50  0000 L CNN
+F 1 "C" H 6125 1750 50  0000 L CNN
+F 2 "Capacitors_SMD:C_0805" H 6138 1700 50  0001 C CNN
+F 3 "" H 6100 1850 50  0001 C CNN
+	1    6100 1850
+	1    0    0    -1
+$EndComp
+$Comp
+L GND #PWR036
+U 1 1 5AB99244
+P 6300 1700
+F 0 "#PWR036" H 6300 1450 50  0001 C CNN
+F 1 "GND" H 6300 1550 50  0000 C CNN
+F 2 "" H 6300 1700 50  0001 C CNN
+F 3 "" H 6300 1700 50  0001 C CNN
+	1    6300 1700
+	1    0    0    -1
+$EndComp
+Wire Wire Line
+	6100 1700 6300 1700
+$Comp
+L Conn_01x02 J10
+U 1 1 5AB996F8
+P 5700 1800
+F 0 "J10" H 5700 1900 50  0000 C CNN
+F 1 "Conn_01x02" H 5700 1600 50  0000 C CNN
+F 2 "Pin_Headers:Pin_Header_Straight_1x02_Pitch2.54mm" H 5700 1800 50  0001 C CNN
+F 3 "" H 5700 1800 50  0001 C CNN
+	1    5700 1800
+	1    0    0    -1
+$EndComp
+Wire Wire Line
+	5500 2100 5500 1900
+$Comp
+L GND #PWR037
+U 1 1 5AB998E1
+P 5400 1800
+F 0 "#PWR037" H 5400 1550 50  0001 C CNN
+F 1 "GND" H 5400 1650 50  0000 C CNN
+F 2 "" H 5400 1800 50  0001 C CNN
+F 3 "" H 5400 1800 50  0001 C CNN
+	1    5400 1800
+	1    0    0    -1
+$EndComp
+Wire Wire Line
+	5500 1800 5400 1800
 $EndSCHEMATC
