File: variable_load.kicad_pcb (KiCad board)
At the start: 2 copper layers, 65 parts, among them J1 Conn_01x04, J2 LEMO, J3 Conn_01x02, J4 GS3, J5 Conn_01x04, J6 Conn_01x04, J7 Conn_01x04, Q1 NTD4858N, U1 DAC5578, U2 LM324, U3 TLV1117-33, U4 PCA9306, U5 adafruit_ft232h, U6 APD123

Commit message: pcb v1
Parts:
- removed C16, C17: C, Capacitors_SMD:C_0805
- moved C9 89.1 mm to (158.0, 71.0)
- moved R9 84.6 mm to (171.0, 60.0)
- moved R5 83.0 mm to (152.0, 71.0)
- moved C8 82.2 mm to (151.0, 75.0)
- moved C10 81.2 mm to (155.0, 71.0), turned to 270 degrees
- moved C7 79.2 mm to (148.0, 75.0)
- moved R4 79.1 mm to (148.0, 70.0), turned to 180 degrees
- moved J2 77.0 mm to (158.0, 79.0)
- moved C1 75.6 mm to (143.0, 63.0), turned to 90 degrees
- moved R3 70.1 mm to (144.0, 77.0), turned to 270 degrees
- moved R6 70.0 mm to (163.0, 70.0)
- moved C2 69.4 mm to (140.0, 63.0)
- moved C18 68.7 mm to (166.0, 58.0), turned to 270 degrees
- moved C23 66.5 mm to (154.0, 48.0)
- moved U1 64.1 mm to (140.0, 70.0), turned to 180 degrees
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Connections:
- C1 pad 2: Earth -> GND
- C10 pad 2: Earth -> GND
- C11 pad 2: Earth -> GND
- C12 pad 2: Earth -> GND
- C14 pad 2: Earth -> GND
- C15 pad 2: Earth -> GND
- C2 pad 2: Earth -> GND
- C20 pad 2: Earth -> GND
- C22 pad 2: Earth -> GND
- C23 pad 2: Earth -> GND
- J2 pad 2: Earth -> GND
- R1 pad 2: Earth -> GND
- R14 pad 2: Earth -> GND
- R3 pad 2: Earth -> GND
- R5 pad 2: Earth -> GND
- R9 pad 1: Earth -> GND
- U1 pad 14: Earth -> GND
- U3 pad 1: Earth -> GND
Routing:
- net /-Vcc: track 10.3 -> 121.7 mm, vias 0 -> 4
- net /SCL_LO: track 0.00 -> 73.7 mm, vias 0 -> 4
- net /VREF: track 0.00 -> 71.1 mm
- net /+Vcc: track 14.7 -> 82.3 mm, vias 0 -> 2
- net /VCC_DAC: track 0.00 -> 59.8 mm, vias 0 -> 2
- net /SDA_LO: track 0.00 -> 56.2 mm, vias 0 -> 2
- net /SDA_HI: track 2.54 -> 56.9 mm
- net /SCL_HI: track 0.00 -> 49.2 mm, vias 0 -> 2
- net Net-(C18-Pad1): track 94.4 -> 46.5 mm, vias 4 -> 0
- net Net-(C19-Pad2): track 84.0 -> 45.6 mm, vias 2 -> 0
- net Earth: track 37.5 -> 0.00 mm
- net /3V3LDO: track 0.00 -> 36.1 mm
- net Net-(C21-Pad2): track 28.1 -> 12.4 mm
- net Net-(R6-Pad1): track 0.00 -> 13.9 mm, vias 0 -> 2
- net /V1: track 0.00 -> 13.1 mm
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
Commit message: pcb v2
Parts:
- moved J7 64.2 mm to (147.0, 38.0), turned to 270 degrees
- moved U5 58.0 mm to (160.0, 63.0), turned to 90 degrees
- moved C6 49.2 mm to (155.0, 39.0), turned to 0 degrees
- moved J6 46.0 mm to (141.0, 27.0)
- moved C5 45.7 mm to (155.0, 36.0), turned to 0 degrees
- moved J1 37.0 mm to (154.0, 27.0)
- moved R17 36.2 mm to (165.0, 71.0), turned to 270 degrees
- moved C25 33.4 mm to (162.0, 71.0)
- moved R3 33.2 mm to (177.0, 73.0)
- moved R18 32.4 mm to (165.0, 67.0)
- moved R19 32.4 mm to (162.0, 67.0)
- moved J2 32.3 mm to (189.0, 70.0)
- moved C3 32.2 mm to (159.0, 36.0), turned to 0 degrees
- moved R1 32.2 mm to (173.0, 73.0), turned to 0 degrees
- moved C7 32.1 mm to (180.0, 72.0)
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Routing:
- net /-Vcc: track 121.7 -> 19.5 mm, vias 4 -> 0
- net /SCL_LO: track 73.7 -> 20.0 mm, vias 4 -> 2
- net /+Vcc: track 82.3 -> 33.9 mm, vias 2 -> 0
- net /SDA_LO: track 56.2 -> 14.5 mm, vias 2 -> 0
- net /VREF: track 71.1 -> 38.0 mm, vias 0 -> 2
- net /SDA_HI: track 56.9 -> 32.2 mm, vias 0 -> 2
- net /3V3LDO: track 36.1 -> 14.9 mm
- net /VCC_DAC: track 59.8 -> 44.6 mm
- net Net-(R12-Pad2): track 23.0 -> 11.7 mm
- net Net-(C24-Pad1): track 33.7 -> 22.6 mm
- net Net-(R3-Pad1): track 6.67 -> 16.1 mm
- net Net-(R1-Pad1): track 4.58 -> 12.2 mm
- net Net-(C19-Pad2): track 45.6 -> 38.5 mm
- net Net-(R20-Pad2): track 5.39 -> 12.0 mm
- net Net-(C18-Pad1): track 46.5 -> 41.8 mm
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- added copper zone on F.Cu, net (none)
Other:
- board outline added: 76.2 x 51 mm

Commit message: pcb v3
Parts:
- added D1: LED, LEDs:LED_1206_HandSoldering, F.Cu at (130.0, 43.0)
- added J8: Conn_01x02, Pin_Headers:Pin_Header_Straight_1x02_Pitch2.54mm, F.Cu at (200.0, 58.0)
- added J9: Conn_01x02, Pin_Headers:Pin_Header_Straight_1x02_Pitch2.54mm, F.Cu at (196.0, 30.0)
- added R22: R, Resistors_SMD:R_0805, F.Cu at (136.0, 44.0)
- added REF**: MountingHole_5mm, Mounting_Holes:MountingHole_5mm, F.Cu at (113.0, 69.0)
- added REF**: MountingHole_5mm, Mounting_Holes:MountingHole_5mm, F.Cu at (113.0, 23.0)
- added REF**: MountingHole_5mm, Mounting_Holes:MountingHole_5mm, F.Cu at (196.0, 69.0)
- added REF**: MountingHole_5mm, Mounting_Holes:MountingHole_5mm, F.Cu at (196.0, 23.0)
- moved U5 34.0 mm to (130.0, 47.0), turned to 180 degrees
- moved C3 19.0 mm to (140.0, 36.0)
- moved C4 19.0 mm to (140.0, 39.0)
- moved C5 19.0 mm to (136.0, 36.0)
- moved C6 19.0 mm to (136.0, 39.0)
- moved J1 19.0 mm to (135.0, 27.0)
- moved J6 19.0 mm to (122.0, 27.0)
- moved J7 19.0 mm to (128.0, 38.0)
- moved Q1 13.6 mm to (159.0, 29.0)
- moved C26 12.2 mm to (128.0, 66.0)
- moved C27 12.2 mm to (128.0, 56.0)
- moved R20 12.2 mm to (128.0, 53.0)
- moved U6 12.2 mm to (128.0, 61.0)
- moved R21 12.0 mm to (132.0, 54.0)
- moved JP2 6.08 mm to (146.0, 57.0)
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Connections:
- C3 pad 1: GND -> Net-(C3-Pad1)
- C5 pad 2: GND -> Net-(C5-Pad2)
- J1 pad 1: /-Vcc -> GND
- J1 pad 3: GND -> /-Vcc
- U1 pad 10: (no net) -> Net-(U1-Pad10)
- U1 pad 11: (no net) -> Net-(U1-Pad11)
- U1 pad 12: (no net) -> Net-(U1-Pad12)
- U1 pad 13: (no net) -> Net-(U1-Pad13)
- U1 pad 5: (no net) -> Net-(U1-Pad5)
- U1 pad 6: (no net) -> Net-(U1-Pad6)
- U1 pad 7: (no net) -> Net-(U1-Pad7)
- U2 pad 10: (no net) -> Net-(U2-Pad10)
- U2 pad 12: (no net) -> Net-(U2-Pad12)
- U2 pad 13: (no net) -> Net-(U2-Pad13)
- U2 pad 14: (no net) -> Net-(U2-Pad14)
- U2 pad 8: (no net) -> Net-(U2-Pad8)
- U2 pad 9: (no net) -> Net-(U2-Pad9)
- U5 pad 1: (no net) -> Net-(U5-Pad1)
- U5 pad 10: (no net) -> Net-(U5-Pad10)
- U5 pad 11: (no net) -> Net-(U5-Pad11)
- U5 pad 12: (no net) -> Net-(U5-Pad12)
- U5 pad 13: (no net) -> Net-(U5-Pad13)
- U5 pad 14: (no net) -> Net-(U5-Pad14)
- U5 pad 15: (no net) -> Net-(U5-Pad15)
- U5 pad 16: (no net) -> Net-(U5-Pad16)
- U5 pad 17: (no net) -> Net-(U5-Pad17)
- U5 pad 18: (no net) -> Net-(U5-Pad18)
- U5 pad 19: (no net) -> Net-(U5-Pad19)
- U5 pad 20: (no net) -> Net-(U5-Pad20)
- U5 pad 6: (no net) -> Net-(U5-Pad6)
- U5 pad 7: (no net) -> Net-(U5-Pad7)
- U5 pad 8: (no net) -> Net-(U5-Pad8)
- U5 pad 9: (no net) -> Net-(U5-Pad9)
Routing:
- net /-Vcc: track 19.5 -> 170.3 mm, vias 0 -> 2
- net /+Vcc: track 33.9 -> 109.8 mm, vias 0 -> 6
- net /VREF: track 38.0 -> 105.4 mm, vias 2 -> 4
- net GND: track 0.14 -> 57.1 mm, vias 0 -> 28
- net /SDA_LO: track 14.5 -> 59.9 mm, vias 0 -> 2
- net /SCL_LO: track 20.0 -> 59.3 mm
- net Net-(C9-Pad1): track 6.41 -> 24.5 mm, vias 0 -> 2
- net Net-(C21-Pad2): track 16.6 -> 33.3 mm
- net Net-(C18-Pad1): track 41.8 -> 56.1 mm
- net Net-(C24-Pad1): track 22.6 -> 35.4 mm
- net /VCC_DAC: track 44.6 -> 56.3 mm, vias 2 -> 4
- net /SDA_HI: track 32.2 -> 39.1 mm, vias 2 -> 4
- net Net-(C19-Pad2): track 38.5 -> 43.7 mm
- net Net-(D1-Pad2): track 0.00 -> 4.05 mm
- net /SCL_HI: track 49.8 -> 53.1 mm, vias 2 -> 6
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- added copper zone on B.Cu, net GND
- added copper zone on F.Cu, net Net-(C18-Pad1)
- added copper zone on F.Cu, net Net-(C24-Pad1)
- removed copper zone on F.Cu, net (none)
Other:
- board size 76.2 x 51 mm -> 96 x 58 mm

Commit message: pcb v4
Parts:
- added G***: LOGO, lbnl_logo:lbnl_logo_small, F.Cu at (112.8, 55.6)
- J7: value Conn_01x04 -> GND
- moved J7 71.9 mm to (199.9, 38.1), turned to 0 degrees
- moved C11 4.77 mm to (183.4, 56.1), turned to 0 degrees
- moved C20 1.82 mm to (182.6, 50.8), turned to 180 degrees
- moved R9 1.70 mm to (183.4, 53.3)
- moved REF** 1.60 mm to (196.8, 70.4)
- moved REF** 1.38 mm to (112.8, 70.4)
- moved ? 0.94 mm to (196.8, 22.6)
- moved ? 0.45 mm to (112.8, 22.6)
- renumbered REF** to ?, U1 to DAC, J6 to I2C, U6 to LDO, J2 to LEMO, J5 to Load, Q1 to MOSFET, U2 to Op-amp, J1 to Power
Connections:
- C26 pad 1: Net-(C26-Pad1) -> /+Vcc
- I2C pad 1: /VREF -> GND
- I2C pad 2: /SCL_LO -> /VREF
- I2C pad 3: GND -> /SCL_LO
- LDO pad 3: Net-(C26-Pad1) -> /+Vcc
Routing:
- net GND: track 57.1 -> 68.4 mm, vias 28 -> 31
- net /VREF: track 105.4 -> 115.7 mm, vias 4 -> 6
- net /+Vcc: track 109.8 -> 119.3 mm
- net /-Vcc: track 170.3 -> 175.4 mm
- net Net-(C19-Pad2): track 43.7 -> 47.9 mm
- net Net-(C26-Pad1): track 3.60 -> 0.00 mm
- net /SCL_LO: track 59.3 -> 57.9 mm, vias 2 -> 4
- net Net-(C18-Pad1): track 56.1 -> 55.5 mm
- net Net-(C24-Pad1): vias 0 -> 2
- net (no net): vias 0 -> 2
- added copper zone on F.Cu, net Net-(C19-Pad2)
- added copper zone on B.Cu, net Net-(C24-Pad1)
Other:
- board size 96 x 58 mm -> 96 x 59.3 mm
- rule pad_to_mask_clearance: 0.2 -> 0
- board text added: "Variable load Neha Santpur 18 Mar 2018"

Commit message: pcb v4
Routing:
- net GND: track 68.4 -> 63.9 mm, vias 31 -> 30
- net (no net): track 0.07 -> 0.25 mm, vias 2 -> 31
- net Net-(U5-Pad13): vias 1 -> 0
- net Net-(U5-Pad11): vias 1 -> 0
- net Net-(C24-Pad1): vias 2 -> 8
Changed lines of the file:
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@@
   (general
     (links 145)
-    (no_connects 1)
+    (no_connects 0)
     (area 106.924988 16.92499 203.075001 76.345001)
     (thickness 1.6)
     (drawings 5)
-    (tracks 532)
+    (tracks 562)
     (zones 0)
     (modules 72)
@@
   (layers
     (0 F.Cu signal)
-    (31 B.Cu signal)
+    (31 B.Cu signal hide)
     (32 B.Adhes user)
     (33 F.Adhes user)
@@
   (gr_line (start 106.999989 17) (end 203 17) (angle 90) (layer Edge.Cuts) (width 0.15))
   (gr_line (start 107 16.999991) (end 107 76.2) (angle 90) (layer Edge.Cuts) (width 0.15))
+  (via (at 162.052 29.972) (size 0.6096) (drill 0.4064) (layers F.Cu B.Cu) (net 0))
+  (via (at 162.052 27.94) (size 0.6096) (drill 0.4064) (layers F.Cu B.Cu) (net 0))
+  (via (at 165.862 26.162) (size 0.6096) (drill 0.4064) (layers F.Cu B.Cu) (net 0))
+  (via (at 163.83 26.162) (size 0.6096) (drill 0.4064) (layers F.Cu B.Cu) (net 0))
+  (via (at 162.052 26.162) (size 0.6096) (drill 0.4064) (layers F.Cu B.Cu) (net 0))
+  (via (at 155.956 29.972) (size 0.6096) (drill 0.4064) (layers F.Cu B.Cu) (net 0))
+  (via (at 155.956 27.94) (size 0.6096) (drill 0.4064) (layers F.Cu B.Cu) (net 0))
+  (via (at 155.956 26.162) (size 0.6096) (drill 0.4064) (layers F.Cu B.Cu) (net 0))
+  (via (at 155.956 24.384) (size 0.6096) (drill 0.4064) (layers F.Cu B.Cu) (net 0))
+  (via (at 163.83 29.972) (size 0.6096) (drill 0.4064) (layers F.Cu B.Cu) (net 0))
+  (via (at 163.83 24.384) (size 0.6096) (drill 0.4064) (layers F.Cu B.Cu) (net 0))
+  (via (at 165.862 29.972) (size 0.6096) (drill 0.4064) (layers F.Cu B.Cu) (net 0))
+  (via (at 153.67 27.94) (size 0.6096) (drill 0.4064) (layers F.Cu B.Cu) (net 0))
+  (via (at 153.67 24.384) (size 0.6096) (drill 0.4064) (layers F.Cu B.Cu) (net 0))
+  (via (at 162.052 22.606) (size 0.6096) (drill 0.4064) (layers F.Cu B.Cu) (net 0))
+  (via (at 157.988 22.606) (size 0.6096) (drill 0.4064) (layers F.Cu B.Cu) (net 0))
+  (via (at 165.862 22.606) (size 0.6096) (drill 0.4064) (layers F.Cu B.Cu) (net 0))
   (via (at 145.796 27.94) (size 0.6096) (drill 0.4064) (layers F.Cu B.Cu) (net 0))
   (via (at 176.276 19.304) (size 0.6096) (drill 0.4064) (layers F.Cu B.Cu) (net 0))
-  (segment (start 142 74.95) (end 141.95 75) (width 0.254) (layer F.Cu) (net 0))
+  (via (at 145.796 19.304) (size 0.6096) (drill 0.4064) (layers F.Cu B.Cu) (net 0))
+  (via (at 176.276 27.94) (size 0.6096) (drill 0.4064) (layers F.Cu B.Cu) (net 0))
+  (via (at 162.052 24.384) (size 0.6096) (drill 0.4064) (layers F.Cu B.Cu) (net 0))
+  (segment (start 164.084 28.448) (end 163.83 28.448) (width 0.254) (layer F.Cu) (net 0))
+  (via (at 163.83 27.94) (size 0.6096) (drill 0.4064) (layers F.Cu B.Cu) (net 0))
+  (via (at 165.862 27.94) (size 0.6096) (drill 0.4064) (layers F.Cu B.Cu) (net 0))
+  (via (at 153.67 29.972) (size 0.6096) (drill 0.4064) (layers F.Cu B.Cu) (net 0))
+  (via (at 153.67 26.162) (size 0.6096) (drill 0.4064) (layers F.Cu B.Cu) (net 0))
+  (via (at 153.67 22.606) (size 0.6096) (drill 0.4064) (layers F.Cu B.Cu) (net 0))
+  (via (at 163.83 22.606) (size 0.6096) (drill 0.4064) (layers F.Cu B.Cu) (net 0))
+  (via (at 160.02 22.606) (size 0.6096) (drill 0.4064) (layers F.Cu B.Cu) (net 0))
+  (via (at 165.862 24.384) (size 0.6096) (drill 0.4064) (layers F.Cu B.Cu) (net 0))
+  (via (at 155.956 22.606) (size 0.6096) (drill 0.4064) (layers F.Cu B.Cu) (net 0))
   (segment (start 162 51) (end 161 51) (width 0.254) (layer F.Cu) (net 1))
   (segment (start 160 54.05) (end 161 55.05) (width 0.254) (layer F.Cu) (net 1))
@@
   (segment (start 180 72) (end 177 72) (width 0.254) (layer F.Cu) (net 1) (status 10))
   (segment (start 168 59.675) (end 167.95 59.725) (width 0.254) (layer F.Cu) (net 1) (status 30))
-  (segment (start 199.898 38.1) (end 197.612 38.1) (width 0.254) (layer F.Cu) (net 2))
-  (via (at 196.342 39.37) (size 0.6096) (drill 0.4064) (layers F.Cu B.Cu) (net 2))
-  (segment (start 197.612 38.1) (end 196.342 39.37) (width 0.254) (layer F.Cu) (net 2))
+  (segment (start 162 70) (end 162.918 70) (width 0.254) (layer F.Cu) (net 2))
+  (via (at 163.576 69.342) (size 0.6096) (drill 0.4064) (layers F.Cu B.Cu) (net 2))
+  (segment (start 162.918 70) (end 163.576 69.342) (width 0.254) (layer F.Cu) (net 2))
   (segment (start 151.85 41.7) (end 151.85 39.92) (width 0.254) (layer F.Cu) (net 2))
   (via (at 151.892 39.878) (size 0.6096) (drill 0.4064) (layers F.Cu B.Cu) (net 2))
@@
   (via (at 131 57) (size 0.6096) (drill 0.4064) (layers F.Cu B.Cu) (net 2))
   (segment (start 130 57) (end 131 57) (width 0.254) (layer F.Cu) (net 2))
-  (segment (start 140.16 69.86) (end 138.14 69.86) (width 0.254) (layer F.Cu) (net 2))
-  (via (at 138 70) (size 0.6096) (drill 0.4064) (layers F.Cu B.Cu) (net 2))
-  (segment (start 138.14 69.86) (end 138 70) (width 0.254) (layer F.Cu) (net 2))
   (segment (start 127 66) (end 127 68) (width 0.254) (layer F.Cu) (net 2))
   (via (at 127 68) (size 0.6096) (drill 0.4064) (layers F.Cu B.Cu) (net 2))
@@
   (segment (start 151.85 44) (end 158.15 44) (width 1.016) (layer F.Cu) (net 13) (status 30))
   (segment (start 158.15 44) (end 162 45) (width 0.254) (layer F.Cu) (net 13) (status 10))
-  (via (at 145.796 19.304) (size 0.6096) (drill 0.4064) (layers F.Cu B.Cu) (net 14))
-  (via (at 176.276 27.94) (size 0.6096) (drill 0.4064) (layers F.Cu B.Cu) (net 14))
+  (via (at 160.02 29.972) (size 0.6096) (drill 0.4064) (layers F.Cu B.Cu) (net 14))
+  (via (at 160.02 26.162) (size 0.6096) (drill 0.4064) (layers F.Cu B.Cu) (net 14))
+  (via (at 157.988 29.972) (size 0.6096) (drill 0.4064) (layers F.Cu B.Cu) (net 14))
+  (via (at 157.988 27.94) (size 0.6096) (drill 0.4064) (layers F.Cu B.Cu) (net 14))
+  (via (at 157.988 26.162) (size 0.6096) (drill 0.4064) (layers F.Cu B.Cu) (net 14))
+  (via (at 160.02 24.384) (size 0.6096) (drill 0.4064) (layers F.Cu B.Cu) (net 14))
+  (via (at 157.988 24.384) (size 0.6096) (drill 0.4064) (layers F.Cu B.Cu) (net 14))
+  (via (at 160.02 27.94) (size 0.6096) (drill 0.4064) (layers F.Cu B.Cu) (net 14))
   (segment (start 191 30) (end 196 30) (width 0.254) (layer F.Cu) (net 14))
   (segment (start 182 27) (end 177.9 27) (width 0.254) (layer F.Cu) (net 14))
@@
   (segment (start 136 43) (end 136 43.05) (width 0.254) (layer F.Cu) (net 30))
   (segment (start 120 54) (end 119.95 54.05) (width 0.254) (layer F.Cu) (net 57) (status 30))
-  (via (at 120 54) (size 0.6096) (drill 0.4064) (layers F.Cu B.Cu) (net 57) (status 30))
   (segment (start 120.05 52) (end 120 52) (width 0.254) (layer F.Cu) (net 58) (status 30))
   (segment (start 120 50) (end 120 49) (width 0.254) (layer B.Cu) (net 59) (status 30))
-  (via (at 120 50) (size 0.6096) (drill 0.4064) (layers F.Cu B.Cu) (net 59) (status 30))
   (zone (net 14) (net_name "Net-(C24-Pad1)") (layer F.Cu) (hatch edge 0.508)
     (connect_pads yes (clearance 0.508))
@@
     )
   )
-  (zone (net 2) (net_name GND) (layer B.Cu) (hatch edge 0.508)
+  (zone (net 14) (net_name "Net-(C24-Pad1)") (layer B.Cu) (hatch edge 0.508)
+    (priority 1)
     (connect_pads yes (clearance 0.508))
     (min_thickness 0.254)
@@
     (polygon
       (pts
-        (xy 107.696 25.4) (xy 143.256 25.4) (xy 143.256 38.862) (xy 202.438 38.862) (xy 202.438 75.692)
-        (xy 107.442 75.692)
+        (xy 178.308 30.988) (xy 144.018 30.988) (xy 144.018 18.034) (xy 178.308 18.034)
       )
     )
   )
-  (zone (net 14) (net_name "Net-(C24-Pad1)") (layer B.Cu) (hatch edge 0.508)
+  (zone (net 2) (net_name GND) (layer B.Cu) (hatch edge 0.508)
     (connect_pads yes (clearance 0.508))
     (min_thickness 0.254)
@@
     (polygon
       (pts
-        (xy 178.308 30.988) (xy 144.018 30.988) (xy 144.018 18.034) (xy 178.308 18.034)
+        (xy 202.438 75.946) (xy 107.442 75.946) (xy 107.442 17.526) (xy 202.438 17.272)
+      )
+    )
+  )
+  (zone (net 0) (net_name "") (layer B.Mask) (hatch edge 0.508)
+    (connect_pads (clearance 0.508))
+    (min_thickness 0.254)
+    (fill yes (arc_segments 16) (thermal_gap 0.508) (thermal_bridge_width 0.508))
+    (polygon
+      (pts
+        (xy 166.624 30.988) (xy 152.4 30.988) (xy 152.4 21.844) (xy 166.624 21.844)
+      )
+    )
+  )
+  (zone (net 0) (net_name "") (layer F.Mask) (hatch edge 0.508)
+    (connect_pads (clearance 0.508))
+    (min_thickness 0.254)
+    (fill yes (arc_segments 16) (thermal_gap 0.508) (thermal_bridge_width 0.508))
+    (polygon
+      (pts
+        (xy 170.688 37.084) (xy 164.084 37.084) (xy 164.084 21.336) (xy 170.688 21.336)
+      )
+    )
+  )
+  (zone (net 0) (net_name "") (layer F.Mask) (hatch edge 0.508)
+    (connect_pads (clearance 0.508))
+    (min_thickness 0.254)
+    (fill yes (arc_segments 16) (thermal_gap 0.508) (thermal_bridge_width 0.508))
+    (polygon
+      (pts
+        (xy 153.924 37.084) (xy 147.32 37.084) (xy 147.32 21.336) (xy 153.924 21.336)
       )
     )

Commit message: pcb v5
Parts:
- added C16: C, Capacitors_SMD:C_0805, F.Cu at (169.9, 57.4)
- added J10: Conn_01x02, Pin_Headers:Pin_Header_Straight_1x02_Pitch2.54mm, F.Cu at (174.8, 53.1)
- moved C21 1.96 mm to (173.0, 50.0)
- renumbered D1 to LED, U5 to USB
Routing:
- net (no net): track 0.25 -> 48.4 mm, vias 31 -> 27
- net Net-(C24-Pad1): track 35.4 -> 42.1 mm
- net Net-(C18-Pad1): track 55.5 -> 49.5 mm
- net Net-(J10-Pad2): track 11.7 -> 15.5 mm
- net Net-(C16-Pad2): track 33.3 -> 35.6 mm
- net GND: track 63.9 -> 65.2 mm, vias 30 -> 31

Commit message: pcb v6
Parts:
- moved C21 3.81 mm to (173.0, 46.2)
- moved C16 2.55 mm to (170.2, 59.9)
- moved J10 2.55 mm to (174.5, 50.5)
- moved R12 0.74 mm to (172.7, 57.1)
Routing:
- net Net-(C24-Pad1): track 42.1 -> 113.6 mm, vias 8 -> 40
- net (no net): track 48.4 -> 0.00 mm, vias 27 -> 0
- net Net-(C18-Pad1): track 49.5 -> 45.7 mm
- net Net-(C16-Pad2): track 35.6 -> 37.6 mm
- net Net-(J10-Pad2): track 15.5 -> 17.1 mm
- net GND: track 65.2 -> 64.4 mm

Commit message: pcb v7
Parts:
- J8 LEMO: renamed from J8
- JP2 SCL: renamed from JP2
- JP3 SDA: renamed from JP3
Routing:
- net /VREF: track 115.7 -> 90.9 mm
- net GND: track 64.4 -> 58.6 mm, vias 31 -> 30
- net /-Vcc: track 175.4 -> 173.0 mm
Other:
- board size 96 x 59.3 mm -> 96 x 59.8 mm
- board text added: "+Vcc"
- board text added: "-Vcc"
- board text added: "GND"
- board text added: "SCL_LO"
- board text added: "SDA_LO"
- board text added: "VREF"
