File: variable_load.kicad_pcb (KiCad board)
At the start: 2 copper layers, 96 x 59.8 mm, 74 parts, among them J10 Conn_01x02, J3 Conn_01x02, J4 GS3, J7 GND, J8 LEMO Conn_01x02, J9 Conn_01x02, U3 TLV1117-33, U4 PCA9306

Commit message: pcb with gerbers
Parts:
- J8: renamed from J8 LEMO
Other:
- board text added: "Variable load Neha Santpur 26 Mar 2018"
- board text removed: "Variable load Neha Santpur 18 Mar 2018"
Changed lines of the file:
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@@
     (links 149)
     (no_connects 1)
-    (area 106.924988 16.92499 203.075001 76.853001)
+    (area 105.307714 12.330999 204.80162 77.487)
     (thickness 1.6)
     (drawings 13)
@@
     (visible_elements FFFFFF7F)
     (pcbplotparams
-      (layerselection 0x00030_80000001)
+      (layerselection 0x010b0_80000001)
       (usegerberextensions false)
       (excludeedgelayer true)
@@
       (outputformat 1)
       (mirror false)
-      (drillshape 1)
+      (drillshape 0)
       (scaleselection 1)
-      (outputdirectory ""))
+      (outputdirectory gerbers/))
   )
   (net 0 "")
@@
     (descr "LEMO connector, EPB.00.250.NTN")
     (fp_text reference LEMO (at 4.93 -0.182 360) (layer F.SilkS)
-      (effects (font (thickness 0.3048)))
+      (effects (font (size 1.27 1.27) (thickness 0.3048)))
     )
     (fp_text value LEMO (at 0 -4.8006 270) (layer Cmts.User)
@@
     (descr "Through hole straight pin header, 1x02, 2.54mm pitch, single row")
     (tags "Through hole pin header THT 1x02 2.54mm single row")
-    (fp_text reference "J8 LEMO" (at 1.168 -5.168 90) (layer F.SilkS)
+    (fp_text reference J8 (at 1.168 -2.628 90) (layer F.SilkS)
       (effects (font (size 1 1) (thickness 0.15)))
     )
@@
     (effects (font (size 0.762 0.762) (thickness 0.1905)))
   )
-  (gr_text "Variable load\nNeha Santpur\n18 Mar 2018\n" (at 112.776 61.214) (layer F.SilkS)
+  (gr_text "Variable load\nNeha Santpur\n26 Mar 2018\n" (at 112.776 61.214) (layer F.SilkS)
     (effects (font (size 1.016 1.016) (thickness 0.1905)))
   )
